File: Ricardo-Hermes.kicad_pcb (KiCad board)
At the start: 4 copper layers, 43 x 63 mm, 145 parts, among them IC2 SX1280, J1 RBUS, J2 USB_C_Receptacle_USB2.0, J3 Conn_01x03_Pin, J4 Conn_01x03_Pin, U1 ESP32-S3, U11 SC4215ASTRT, U12 SKY66112-11, U13 DEA202450BT-1213C1, U2 SN65HVD230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

Commit message: Finishing touches without BOM
Parts:
- removed U13, U6: DEA202450BT-1213C1, iclr:DEA-4_2P0X1P25
- added C77: 0.4 pF, Capacitor_SMD:C_0402_1005Metric, F.Cu at (145.8, 113.9)
- added C78: 1.2 pF, Capacitor_SMD:C_0402_1005Metric, F.Cu at (145.8, 116.8)
- added C79: 0.5 pF, Capacitor_SMD:C_0402_1005Metric, F.Cu at (147.3, 118.3)
- added C80: 1.2 pF, Capacitor_SMD:C_0402_1005Metric, F.Cu at (145.8, 119.8)
- added L7: DET_LATER, Inductor_SMD:L_0402_1005Metric, F.Cu at (146.3, 115.4)
- added L8: 0.5 pF, Inductor_SMD:L_0402_1005Metric, F.Cu at (146.3, 118.3)
- moved C71 3.44 mm to (151.9, 119.2)
- moved U12 3.44 mm to (146.6, 122.4)
- moved C61 3.44 mm to (149.5, 126.6)
- moved C65 3.44 mm to (148.7, 125.6)
- moved C66 3.44 mm to (149.4, 121.5)
- moved C68 3.44 mm to (150.4, 120.5)
- moved C70 3.44 mm to (149.0, 124.1)
- moved C73 3.44 mm to (150.0, 124.1)
- moved C74 3.44 mm to (152.0, 123.8)
- moved FB_R1 3.44 mm to (153.1, 121.5)
- moved VAA_TP1 3.44 mm to (154.9, 123.5)
- moved ANT1 2.00 mm to (145.8, 131.5)
- moved G*** 2.00 mm to (130.2, 132.2)
- moved H3 2.00 mm to (121.7, 132.6)
- moved H4 2.00 mm to (157.7, 132.6)
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Connections:
- IC2 pad 22: RF_OUT_T -> Net-(IC2-RFIO)
- U12 pad 6: Net-(U12-ANT2) -> Net-(ANT2-In)
- U12 pad 8: Net-(U12-ANT1) -> Net-(ANT1-In)
Routing:
- net CPS: track 36.8 -> 43.0 mm
- net GND: track 330.7 -> 336.8 mm, vias 201 -> 205
- net +VDC: track 35.4 -> 40.9 mm
- net CHL: track 32.9 -> 38.1 mm
- net CTX: track 34.0 -> 38.4 mm
- net Net-(U12-ANT2): track 3.99 -> 0.00 mm
- net VAA: track 51.0 -> 54.7 mm
- net RF_RST: track 29.8 -> 33.4 mm
- net Net-(ANT2-In): track 2.51 -> 5.95 mm
- net Net-(ANT1-In): track 5.96 -> 9.30 mm
- net Net-(U12-ANT1): track 3.12 -> 0.00 mm
- net Net-(C78-Pad1): track 0.00 -> 2.97 mm
- net /CAN_TX: track 35.3 -> 33.0 mm
- net Net-(IC2-RFIO): track 0.00 -> 2.16 mm
- net RF_OUT_T: track 4.74 -> 3.16 mm
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Other:
- board size 43 x 63 mm -> 43 x 65 mm
- board text added: "I had to do this ugly shit because kicad 9 kinda broke zone fills..."
- board text added: "We also have various errors on differential pair spacing, was done intentionally to make routing neater"
- board text removed: "Check current for vdd pins! 0403 can only handle 1/8W, might have to move to chunkier stuff."

Commit message: finishing changes
Parts:
- removed the G*** at (130.2, 132.2)
- added R7: 499R, Resistor_SMD:R_0402_1005Metric, F.Cu at (129.3, 121.5)
- added UART2: Conn_01x03, Connector_PinHeader_2.54mm:PinHeader_1x03_P2.54mm_Vertical, F.Cu at (125.0, 128.0)
- DIO3_D1: value GREEN_LED -> BLUE_LED
- FB_R1: value FerriteBead_Small -> FB
- L7: value DET_LATER -> 3.0 nH
- POWER UART: renamed from POWER_UART1; footprint Connector_PinHeader_2.54mm:PinHeader_1x02_P2.54mm_Vertical -> Connector_PinHeader_2.54mm:PinHeader_1x01_P2.54mm_Vertical
- R31, R32, R33, R34: value 20-100 -> 50
- RXD_1_RDIO: renamed from RXD_1; value GREEN_LED -> ORANGE_LED
- moved R6 4.83 mm to (133.2, 123.9), turned to 90 degrees
- moved UART1 2.03 mm to (126.6, 124.0)
- moved C27 1.03 mm to (135.4, 83.2)
- moved POWER UART 0.96 mm to (130.1, 118.5)
- moved BBOUT_TP1 0.53 mm to (126.4, 74.2)
- moved TXLED1 0.51 mm to (129.3, 122.5)
- moved R2 0.51 mm to (129.3, 123.5)
- moved R17 0.44 mm to (139.9, 82.2)
- moved R16 0.44 mm to (138.0, 82.2)
- moved C24 0.44 mm to (139.2, 73.8)
- moved C25 0.44 mm to (137.0, 73.8)
- moved C26 0.44 mm to (136.2, 82.1)
- moved U5 0.44 mm to (138.0, 78.0)
- moved L2 0.24 mm to (136.9, 97.5)
- moved DIO3 0.13 mm to (146.6, 101.0)
- renumbered ANT1 to ANT_SMA1, ANT2 to ANT_UFL1, J3 to PWR_AMP, TXD_1 to TXD_1_RDIO, R35 to VCC_SX1
Connections:
- R6 pad 1: /TXD -> /TXD_ESP
- U1 pad 47: unconnected-(U1-MTDI/JTAG/GPIO41-Pad47) -> Net-(U1-MTDI/JTAG/GPIO41)
- U1 pad 48: unconnected-(U1-MTMS/JTAG/GPIO42-Pad48) -> /RXD
- U1 pad 50: /RXD -> /RXD_ESP
Routing:
- net /RXD_ESP: track 0.00 -> 37.3 mm, vias 0 -> 1
- net Net-(U1-MTDI/JTAG/GPIO41): track 0.00 -> 34.0 mm, vias 0 -> 2
- net GND: track 336.8 -> 326.6 mm, vias 205 -> 203
- net /TXD_ESP: track 0.00 -> 6.07 mm
- net Net-(J4-Pin_2): track 15.0 -> 16.9 mm
- net /TXD: track 5.47 -> 3.66 mm
- net Net-(U1-U0TXD/PROG/GPIO43): track 33.1 -> 31.4 mm
- net +3V3: track 128.9 -> 127.7 mm
- net /RXD: track 37.1 -> 36.1 mm
- net +VDC: track 40.9 -> 40.5 mm, vias 3 -> 1
- added copper zone on F.Cu, net +VDC
- removed copper zone on F.Cu, net VBUS
Other:
- board text removed: "I had to do this ugly shit because kicad 9 kinda broke zone fills..."
- board text removed: "JLCJLCJLCJLC"
- board text removed: "We also have various errors on differential pair spacing, was done intentionally to make routing neater"

Commit message: Prod Files
Parts:
- C50, C51: value C_Small -> 15pF
- FB_R1: value FB -> C3011209
- L8: value 0.5 pF -> 2.5nH
- POWER_UART1: renamed from POWER UART
- Y3: value Crystal_GND24 -> C3034316
- renumbered PWR_AMP to J3, RXD_1_RDIO to RXD_1_R1, TXD_1_RDIO to TXD_1_R1

Commit message: Final manu files
Needs to be looked over
Parts:
- added REF**: Square of knowledge, Ky:Square_Of_Knowledge_QRCODE, F.Cu at (140.4, 122.5)

Commit message: Minor fix
Routing:
- net GND: track 326.6 -> 336.3 mm
